File: Schematics/laser_driver.kicad_sch (KiCad schematic)
At the start: 52 parts, among them J1 Rows, J2 Cols, J3 To CPU, Q1 BS250, Q10 2N7000, Q11 2N7000, Q12 2N7000, Q2 BS250, Q3 BS250, Q4 BS250, Q5 BS250, Q6 BS250, Q7 2N7000, Q8 2N7000, Q9 2N7000, U1 74HC138, U2 74HC138, U3 74LS04

Commit message: Lopts and  lots of changes for new body and circuitry
Parts:
- C1, C2, C3: footprint (none) -> Capacitor_THT:C_Rect_L10.0mm_W3.0mm_P7.50mm_FKS3_FKP3
- J1: value Rows -> Anodes; footprint (none) -> Connector_PinHeader_2.54mm:PinHeader_1x06_P2.54mm_Vertical
- J2: value Cols -> Cathodes; footprint (none) -> Connector_PinHeader_2.54mm:PinHeader_1x06_P2.54mm_Vertical
- J3: footprint (none) -> Connector_PinHeader_2.54mm:PinHeader_1x09_P2.54mm_Vertical
- R1, R10, R11, R12, R13, R14, R15, R16, R17, R18, R19, R2, R20, R21, R22, R23, R24, R25, R26, R27, R28, R29, R3, R30, R31, R4, R5, R6, R7, R9: footprint (none) -> Resistor_THT:R_Axial_DIN0204_L3.6mm_D1.6mm_P7.62mm_Horizontal
- R8: value R_Small -> 100k; footprint (none) -> Resistor_THT:R_Axial_DIN0204_L3.6mm_D1.6mm_P7.62mm_Horizontal
- U1, U2: footprint (none) -> Package_DIP:DIP-16_W10.16mm
- U3: footprint (none) -> Package_DIP:DIP-14_W7.62mm_Socket
Connections:
- net +3.3V: no longer Q1.3 (S), Q2.3 (S), Q3.3 (S), Q4.3 (S), Q5.3 (S), Q6.3 (S), R10.1, R11.1, R12.1, R13.1, R8.1, R9.1, U1.16 (VCC)
- net GND: no longer R26.2, R27.2, R28.2, R29.2, R30.2, R31.1
- net at R7.1: now also U1.10 (~{Y5}); no longer U3.12
- net at R31.2, U3.13: now also U2.10 (~{Y5}); no longer U1.10 (~{Y5})
- net at R30.1, U3.11: now also U2.11 (~{Y4}); no longer U1.11 (~{Y4})
- net at R29.1, U3.9: now also U2.12 (~{Y3}); no longer U1.12 (~{Y3})
- net at R28.1, U3.5: now also U2.13 (~{Y2}); no longer U1.13 (~{Y2})
- net at R27.1, U3.3: now also U2.14 (~{Y1}); no longer U1.14 (~{Y1})
- net at R26.1, U3.1: now also U2.15 (~{Y0}); no longer U1.15 (~{Y0})
- net at R5.1: now also U1.12 (~{Y3}); no longer U3.8
- net at R6.1: now also U1.11 (~{Y4}); no longer U3.10
- net at R3.1: now also U1.14 (~{Y1}); no longer U3.4
- net at R17.1: now also U3.8; no longer U2.12 (~{Y3})
- net at R2.1: now also U1.15 (~{Y0}); no longer U3.2
- net at R15.1: now also U3.4; no longer U2.14 (~{Y1})
- net at R18.1: now also U3.10; no longer U2.11 (~{Y4})
- net at R4.1: now also U1.13 (~{Y2}); no longer U3.6
- net at R19.1: now also U3.12; no longer U2.10 (~{Y5})
- net at R16.1: now also U3.6; no longer U2.13 (~{Y2})
- net at R14.1: now also U3.2; no longer U2.15 (~{Y0})
- new net: R26.2, R27.2, R28.2, R29.2, R30.2, R31.1
- new net V_LSR: Q1.3 (S), Q2.3 (S), Q3.3 (S), Q4.3 (S), Q5.3 (S), Q6.3 (S), R10.1, R11.1, R12.1, R13.1, R8.1, R9.1, U1.16 (VCC)
Other:
- title: EHarp2 Laser Driver board -> EHarp2 laser driver section
- moved on the sheet: J1, J2, Q1, Q10, Q11, Q12, Q2, Q3, Q4, Q5, Q6, Q7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
