File: Schematics/eHarp_sschematics_mainboard.kicad_sch (KiCad schematic)
At the start: 38 parts, among them J1 Display, J2 Columns, J3 Rows, J4 MIDI Jack, J5 MIDI Controls, J6 Sustain Pedal, J7 Power, Q1 2N3904, Q2 2N3904, Q3 2N3904, Q4 2N3904, Q5 2N3904, Q6 2N3904, U1 Pico, U3 74HC4051, U4 74HC4051, U5 LM393

Commit message: New menu system; new code for baseline management, updated schematics
Parts:
- removed C1, C2: 0.1 uF, Capacitor_THT:C_Rect_L9.0mm_W2.5mm_P7.50mm_MKT, symbol Device:C_Small
- removed J2: Columns, Connector_PinHeader_2.54mm:PinHeader_1x06_P2.54mm_Vertical, symbol Connector:Conn_01x06_Male
- removed J3: Rows, Connector_PinHeader_2.54mm:PinHeader_1x06_P2.54mm_Vertical, symbol Connector:Conn_01x06_Male
- removed Q1, Q2, Q3, Q4, Q5, Q6: 2N3904, Package_TO_SOT_THT:TO-92_Inline, symbol Transistor_BJT:2N3904
- removed R1, R2, R23, R3, R4, R5, R6: 10k, Resistor_THT:R_Axial_DIN0204_L3.6mm_D1.6mm_P7.62mm_Horizontal, symbol Device:R_Small
- removed R19: 10k, Potentiometer_THT:Potentiometer_Bourns_3266W_Vertical, symbol Device:R_Trim
- removed U3, U4: 74HC4051, Package_DIP:DIP-16_W7.62mm, symbol 74xx:74HC4051
- removed U5: LM393, Package_DIP:DIP-8_W7.62mm, symbol Comparator:LM393
- added C4, C5, C6: 0.1uF, Capacitor_THT:C_Rect_L10.0mm_W3.0mm_P7.50mm_FKS3_FKP3, symbol Device:C_Small
- added C7: 2.2nF, Capacitor_THT:C_Rect_L10.0mm_W3.0mm_P7.50mm_FKS3_FKP3, symbol Device:C_Small
- added C8: 10uF, Capacitor_THT:CP_Radial_D10.0mm_P2.50mm, symbol Device:C_Polarized_Small
- added J10: Cathodes, Connector_PinHeader_2.54mm:PinHeader_1x06_P2.54mm_Vertical, symbol Connector:Conn_01x06_Pin
- added J8: Sensor, Connector_PinHeader_2.54mm:PinHeader_1x02_P2.54mm_Vertical, symbol Connector:Conn_01x02_Male
- added J9: Anodes, Connector_PinHeader_2.54mm:PinHeader_1x06_P2.54mm_Vertical, symbol Connector:Conn_01x06_Pin
- added Q1, Q2, Q3, Q4, Q5, Q6: BS250, Package_TO_SOT_THT:TO-92_Inline, symbol Transistor_FET:BS250
- added Q10, Q11, Q12, Q7, Q8, Q9: 2N7000, Package_TO_SOT_THT:TO-92_Inline, symbol Transistor_FET:2N7000
- added R10, R11, R12, R24, R37, R38, R39, R40, R41, R42, R8, R9: 220, Resistor_THT:R_Axial_DIN0204_L3.6mm_D1.6mm_P7.62mm_Horizontal, symbol Device:R_Small
- added R19, R25, R32, R33, R34, R35, R36, R43, R44, R45, R46, R47, R48: 100k, Resistor_THT:R_Axial_DIN0204_L3.6mm_D1.6mm_P7.62mm_Horizontal, symbol Device:R_Small
- added R26, R27, R28, R29, R30, R31, R7: 10k, Resistor_THT:R_Axial_DIN0204_L3.6mm_D1.6mm_P7.62mm_Horizontal, symbol Device:R_Small
- added RV1: 50k, Potentiometer_THT:Potentiometer_Vishay_T93YA_Vertical, symbol Device:R_Potentiometer_Trim
- added U2, U3: 74HC138, Package_DIP:DIP-16_W10.16mm, symbol 74xx:74HC138
- added U4: 74HC04, Package_DIP:DIP-14_W7.62mm, symbol 74xx:74HC04
- added U5: MCP602, Package_DIP:CERDIP-8_W7.62mm_SideBrazed, symbol Amplifier_Operational:MCP602
- added U6: LM393, Package_DIP:CERDIP-8_W7.62mm_SideBrazed, symbol Comparator:LM393
- added U7: 74LS04, Package_DIP:DIP-14_W7.62mm, symbol 74xx:74LS04
- R13, R15, R17, R18: value 82k -> 10k
- R14: value 82k -> 100k
- R16: value 82k -> 1M
- R20: value 10k -> 470k
Connections:
- net +3V3: now also R13.2
- net GND: now also R15.1, C4.1, C5.1, C6.2, C8.2, J8.2 (Pin_2), Q10.1 (S), Q11.1 (S), Q12.1 (S), Q7.1 (S), Q8.1 (S), Q9.1 (S), R43.2, R44.2, R45.2, R46.2, R47.2, R48.2, R7.1, RV1.3, U2.4 (~{E0}), U2.5 (~{E1}), U2.8 (GND), U3.4 (~{E0}), U3.5 (~{E1}), U3.8 (GND), U4.7 (GND), U5.4 (V-), U6.4 (V-); no longer R13.2, R14.2, R15.2, R16.2, R17.2, R18.2, R20.1
- net at U1.10 (GPIO7): now also U3.2 (A1)
- net at U1.11 (GPIO8): now also U3.3 (A2)
- net at U1.12 (GPIO9): now also R7.2, U2.6 (E2), U3.6 (E2)
- net at U1.14 (GPIO10): now also U2.1 (A0)
- net at U1.15 (GPIO11): now also U2.2 (A1)
- net at U1.16 (GPIO12): now also U2.3 (A2)
- net at U1.21 (GPIO16): now also R22.2
- net at U1.22 (GPIO17): now also R13.1, U6.1
- net at U1.24 (GPIO18): now also R18.2
- net at U1.25 (GPIO19): no longer R22.2
- net at U1.31 (GPIO26_ADC0): now also R14.1, C7.2, U5.7, U6.3 (+)
- net at U1.9 (GPIO6): now also U3.1 (A0)
- net +3.3V: now reaches R20.2
- net +3.3V: now also C5.2, C6.1, RV1.1, U3.16 (VCC), U4.14 (VCC), U5.8 (V+), U6.8 (V+)
- net at R18.1: now also R17.2, C8.1
- net at R16.1: now also U5.1, U5.5 (+)
- net at R17.1: now also U5.3 (+)
- new net: Q9.2 (G), R39.2, R45.1
- new net: J10.3 (Pin_3), Q9.3 (D)
- new net: J8.1 (Pin_1), R19.2, R20.1
- new net: R38.1, U7.4
- new net: Q8.2 (G), R38.2, R44.1
- new net: R28.1, U3.13 (~{Y2}), U7.5
- new net: R39.1, U7.6
- new net: R16.2, R19.1, U5.2 (-)
- new net: C7.1, R14.2, R15.2, U5.6 (-)
- new net: R42.1, U7.12
- new net: R31.2, U3.10 (~{Y5}), U7.13
- new net: J10.1 (Pin_1), Q7.3 (D)
- new net: J10.2 (Pin_2), Q8.3 (D)
- new net: J10.4 (Pin_4), Q10.3 (D)
- new net: J10.5 (Pin_5), Q11.3 (D)
- new net: J10.6 (Pin_6), Q12.3 (D)
- new net: R11.1, U2.12 (~{Y3})
- new net: Q4.2 (G), R11.2, R33.2
- new net: Q11.2 (G), R41.2, R47.1
- new net: J9.6 (Pin_6), Q6.1 (D)
- new net: Q6.2 (G), R24.2, R25.2
- new net: R26.2, R27.2, R28.2, R29.2, R30.2, R31.1
- new net: R40.1, U7.8
- new net: Q10.2 (G), R40.2, R46.1
- new net: R41.1, U7.10
- new net: Q3.2 (G), R10.2, R34.2
- new net: R30.1, U3.11 (~{Y4}), U7.11
- new net: R29.1, U3.12 (~{Y3}), U7.9
- new net: R27.1, U3.14 (~{Y1}), U7.3
- new net: R26.1, U3.15 (~{Y0}), U4.1
- new net: R37.1, U4.2
- new net: Q7.2 (G), R37.2, R43.1
- new net: J9.3 (Pin_3), Q3.1 (D)
- new net: Q2.2 (G), R35.2, R9.2
- new net: R10.1, U2.13 (~{Y2})
- new net: Q1.2 (G), R36.2, R8.2
- new net: J9.1 (Pin_1), Q1.1 (D)
- new net: J9.2 (Pin_2), Q2.1 (D)
- new net: J9.4 (Pin_4), Q4.1 (D)
- new net: J9.5 (Pin_5), Q5.1 (D)
- new net: Q12.2 (G), R42.2, R48.1
- new net: Q5.2 (G), R12.2, R32.2
- new net: RV1.2, U6.2 (-)
- new net: R24.1, U2.10 (~{Y5})
- new net: R8.1, U2.15 (~{Y0})
- new net: R12.1, U2.11 (~{Y4})
- new net: R9.1, U2.14 (~{Y1})
- new net 3.3v: C4.2, Q1.3 (S), Q2.3 (S), Q3.3 (S), Q4.3 (S), Q5.3 (S), Q6.3 (S), R25.1, R32.1, R33.1, R34.1, R35.1, R36.1, U2.16 (VCC)
